File: LF_4.0 - 26nat/KiCad/LF_CB_modular_v1/LF_CB_modular_v1.kicad_pcb (KiCad board)
At the start: 2 copper layers, 29 parts, among them J1 Conn_QTR16, J10 Conn_01x02, J11 Conn_01x10, J2 Conn_Arducam_MEGA_3mpx, J3 Conn_TB6612FNG_IC, J4 Conn_01x01, J5 Conn_01x01, J6 Conn_01x01, J8 Conn_01x01, J9 Conn_01x01, M1 Motor_DC, M2 Motor_DC, Q2 IRLZ44N, SW1 SW_SPDT, U1 Teensy4.1, U2 LM7805_TO220, U3 LM2596T-ADJ

Commit message: redesigned power module
Parts:
- removed BT2: Battery_Cell, Connector_AMASS:AMASS_XT60PW-M_1x02_P7.20mm_Horizontal
- removed C1: C_Polarized_100u/25V, Capacitor_THT:CP_Radial_D6.3mm_P2.50mm
- removed C2: C_Polarized_220u/16V, Capacitor_THT:CP_Radial_D8.0mm_P3.50mm
- removed C3, C4: C_100n, Capacitor_THT:C_Disc_D3.8mm_W2.6mm_P2.50mm
- removed D1: LED, LED_THT:LED_D5.0mm
- removed D2: 1N5822, Diode_THT:D_DO-201AD_P15.24mm_Horizontal
- removed J5: Conn_01x01, Connector_PinSocket_2.54mm:PinSocket_1x01_P2.54mm_Vertical
- removed L1: L, Inductor_THT:L_Radial_D10.0mm_P5.00mm_Neosid_SD12k_style3
- removed Q2: IRLZ44N, Package_TO_SOT_THT:TO-220-3_Vertical
- removed R1: R_10k, Resistor_THT:R_Axial_DIN0204_L3.6mm_D1.6mm_P7.62mm_Horizontal
- removed R2: R_150, Resistor_THT:R_Axial_DIN0204_L3.6mm_D1.6mm_P7.62mm_Horizontal
- removed R3: R_1k, Resistor_THT:R_Axial_DIN0204_L3.6mm_D1.6mm_P7.62mm_Horizontal
- removed R4: R_3k9, Resistor_THT:R_Axial_DIN0204_L3.6mm_D1.6mm_P7.62mm_Horizontal
- removed SW1: SW_SPDT, Connector_JST:JST_XH_B2B-XH-A_1x02_P2.50mm_Vertical
- removed U2: LM7805_TO220, Package_TO_SOT_THT:TO-220-3_Vertical
- removed U3: LM2596T-ADJ, Package_TO_SOT_THT:TO-220-5_P3.4x3.7mm_StaggerOdd_Lead3.8mm_Vertical
- J4: value Conn_01x01 -> Conn_01x02; footprint Connector_PinSocket_2.54mm:PinSocket_1x01_P2.54mm_Vertical -> Connector_PinSocket_2.54mm:PinSocket_1x02_P2.54mm_Vertical
- moved J4 60.9 mm to (66.0, 134.8), turned to 180 degrees
- moved J1 4.42 mm to (67.3, 140.5)
Connections:
- J4 pad 1: Net-(J1-EVN) -> Net-(J1-ODD)
Routing:
- net Net-(J1-RC08): track 0.00 -> 55.6 mm
- net Net-(J1-RC06): track 0.00 -> 48.6 mm
- net Net-(J1-RC10): track 0.00 -> 48.6 mm
- net Net-(J1-RC12): track 0.00 -> 41.5 mm
- net Net-(J1-RC04): track 0.00 -> 41.5 mm
- net Net-(J1-RC14): track 0.00 -> 34.4 mm
- net Net-(J1-RC02): track 0.00 -> 34.4 mm
- net Net-(J3-AO1): track 0.00 -> 33.7 mm
- net Net-(J3-AO2): track 0.00 -> 28.0 mm
- net Net-(J1-RC16): track 0.00 -> 27.4 mm
- net Net-(J1-EVN): track 0.00 -> 20.8 mm
- net Net-(J1-RC01): track 0.00 -> 16.5 mm
- net Net-(J3-BO1): track 0.00 -> 16.0 mm
- net Net-(J1-RC03): track 0.00 -> 15.2 mm
- net Net-(J3-BO2): track 0.00 -> 15.1 mm
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
Commit message: started DPS
Parts:
- removed J6: Conn_01x01, Connector_PinSocket_2.54mm:PinSocket_1x01_P2.54mm_Vertical
- added BT2: Battery_Cell, Connector_AMASS:AMASS_XT60PW-M_1x02_P7.20mm_Horizontal, F.Cu at (91.0, 50.1)
- added C1: C_1u, Capacitor_THT:C_Disc_D5.0mm_W2.5mm_P5.00mm, F.Cu at (56.2, 49.8)
- added C2: C_Polarized_47u, Capacitor_THT:CP_Radial_D6.3mm_P2.50mm, F.Cu at (51.2, 48.9)
- added C3: C_100n, Capacitor_THT:C_Disc_D4.3mm_W1.9mm_P5.00mm, F.Cu at (72.2, 62.8)
- added D1: LED, LED_THT:LED_D5.0mm, F.Cu at (77.2, 51.8)
- added HS1: Heatsink_Pad, Linefollower:Heatsink_HS-123-25_TO220_STONECOLD, F.Cu at (53.6, 60.8)
- added Q1: IRF4905, Package_TO_SOT_THT:TO-220-3_Vertical, F.Cu at (84.1, 51.8)
- added R1: R_10k, Resistor_THT:R_Axial_DIN0204_L3.6mm_D1.6mm_P7.62mm_Horizontal, F.Cu at (87.1, 53.1)
- added R2: R_1k, Resistor_THT:R_Axial_DIN0204_L3.6mm_D1.6mm_P7.62mm_Horizontal, F.Cu at (77.2, 54.8)
- added R3: R_33k, Resistor_THT:R_Axial_DIN0204_L3.6mm_D1.6mm_P7.62mm_Horizontal, F.Cu at (70.7, 45.2)
- added R4: R_10k, Resistor_THT:R_Axial_DIN0204_L3.6mm_D1.6mm_P7.62mm_Horizontal, F.Cu at (67.2, 54.8)
- added SW1: SW_SPDT, Connector_JST:JST_XH_B2B-XH-A_1x02_P2.50mm_Vertical, F.Cu at (85.2, 57.8)
- added U2: LM7805_TO220, Package_TO_SOT_THT:TO-220-3_Vertical, F.Cu at (56.2, 52.8)
- moved J1 26.2 mm to (92.3, 132.7)
- moved M2 26.2 mm to (47.9, 98.9)
- moved J10 26.2 mm to (65.7, 91.3)
- moved J11 26.2 mm to (91.1, 76.0)
- moved J3 26.2 mm to (45.4, 73.5)
- moved J4 26.2 mm to (91.0, 127.0)
- moved J8 26.2 mm to (65.7, 70.9)
- moved J9 26.2 mm to (65.7, 106.5)
- moved M1 26.2 mm to (47.9, 109.0)
- moved U1 26.2 mm to (78.4, 97.6)
- moved J2 26.2 mm to (58.0, 109.0)
Connections:
- U1 pad 33: Net-(J6-Pin_1) -> /BATT_SENSE
Routing:
- net /5V: track 0.00 -> 75.7 mm
- net /6V: track 0.00 -> 62.3 mm
- net /3V3: track 0.00 -> 53.0 mm
- net Net-(BT2-+): track 0.00 -> 9.81 mm
- net /BATT_SENSE: track 0.00 -> 9.78 mm
- net Net-(Q1-G): track 0.00 -> 8.98 mm
- net Net-(J6-Pin_1): track 5.08 -> 0.00 mm
- net Net-(D1-K): track 0.00 -> 3.00 mm
- added copper zone on F.Cu, net /GND

Commit message: power modul finishing
Parts:
- added C4: C_100n, Capacitor_THT:C_Disc_D4.3mm_W1.9mm_P5.00mm, F.Cu at (56.2, 45.0)
- added C5: C_100n, Capacitor_THT:C_Disc_D4.3mm_W1.9mm_P5.00mm, F.Cu at (51.1, 44.5)
- added JW1: Cam_SCK, Linefollower:Jumper_pin, F.Cu at (83.0, 101.4)
- added JW2: Cam_SCK, Linefollower:Jumper_pin, F.Cu at (61.0, 104.0)
- added JW3: 3V3, Linefollower:Jumper_pin, F.Cu at (91.0, 130.0)
- added JW4: 3V3, Linefollower:Jumper_pin, F.Cu at (74.0, 104.0)
- U2: value LM7805_TO220 -> LM2940CT-5.0 _TO220
- moved C2 5.27 mm to (46.0, 48.0)
- moved C1 2.82 mm to (59.0, 50.0)
- moved HS1 0.75 mm to (53.6, 60.0)
Connections:
- BT2 pad : (no net) -> /GND
- J1 pad 3: /3V3 -> Net-(JW3-Pin_1)
- J1 pad 4: /3V3 -> Net-(JW3-Pin_1)
- J2 pad 3: /Cam_SCK -> Net-(J2-SCK)
- U1 pad 35: /Cam_SCK -> Net-(JW1-Pin_1)
- U1 pad 46: /3V3 -> unconnected-(U1-3V3-Pad46)
Routing:
- net /BATT_SENSE: track 9.78 -> 69.8 mm
- net /5V: track 75.7 -> 88.8 mm
- net Net-(JW3-Pin_1): track 0.00 -> 5.74 mm
- net /3V3: track 53.0 -> 56.3 mm
- net Net-(JW1-Pin_1): track 0.00 -> 2.99 mm
- net Net-(J2-SCK): track 0.00 -> 2.95 mm
Other:
- board outline added: 60 x 100 mm
