File: LF_4.0 - 26nat/KiCad/LF_CB_modular_v1/LF_CB_modular_v1.kicad_sch (KiCad schematic)
At the start: 29 parts, among them J1 Conn_QTR16, J10 Conn_01x02, J11 Conn_01x10, J2 Conn_Arducam_MEGA_3mpx, J3 Conn_TB6612FNG_IC, J4 Conn_01x01, J5 Conn_01x01, J6 Conn_01x01, J8 Conn_01x01, J9 Conn_01x01, M1 Motor_DC, M2 Motor_DC, Q2 IRLZ44N, SW1 SW_SPDT, U1 Teensy4.1, U2 LM7805_TO220, U3 LM2596T-ADJ

Commit message: redesigned power module
Parts:
- removed C1: C_Polarized_100u/25V, Capacitor_THT:CP_Radial_D6.3mm_P2.50mm, symbol Device:C_Polarized
- removed C4: C_100n, Capacitor_THT:C_Disc_D3.8mm_W2.6mm_P2.50mm, symbol Device:C
- removed D2: 1N5822, Diode_THT:D_DO-201AD_P15.24mm_Horizontal, symbol Diode:1N5822
- removed J4, J5, J6: Conn_01x01, Connector_PinSocket_2.54mm:PinSocket_1x01_P2.54mm_Vertical, symbol Connector_Generic:Conn_01x01
- removed L1: L, Inductor_THT:L_Radial_D10.0mm_P5.00mm_Neosid_SD12k_style3, symbol Device:L
- removed Q2: IRLZ44N, Package_TO_SOT_THT:TO-220-3_Vertical, symbol Transistor_FET:IRLZ44N
- removed U3: LM2596T-ADJ, Package_TO_SOT_THT:TO-220-5_P3.4x3.7mm_StaggerOdd_Lead3.8mm_Vertical, symbol Regulator_Switching:LM2596T-ADJ
- added C1: C_1u, symbol Device:C
- added J4: Conn_01x02, Connector_PinSocket_2.54mm:PinSocket_1x02_P2.54mm_Vertical, symbol Connector_Generic:Conn_01x02
- added Q1: IRF4905, Package_TO_SOT_THT:TO-220-3_Vertical, symbol Transistor_FET:IRF4905
- C2: value C_Polarized_220u/16V -> C_Polarized_47u; footprint Capacitor_THT:CP_Radial_D8.0mm_P3.50mm -> (none)
- C3: footprint Capacitor_THT:C_Disc_D3.8mm_W2.6mm_P2.50mm -> (none)
- R2: value R_150 -> R_1k
- R3: value R_1k -> R_33k; footprint Resistor_THT:R_Axial_DIN0204_L3.6mm_D1.6mm_P7.62mm_Horizontal -> (none)
- R4: value R_3k9 -> R_10k; footprint Resistor_THT:R_Axial_DIN0204_L3.6mm_D1.6mm_P7.62mm_Horizontal -> (none)
Connections:
- net 5V: now also C2.1; no longer C3.1
- net 6V: now also D1.2 (A), R3.1, C1.1, Q1.2 (D); no longer C2.1, R4.1
- net GND: now also BT2.2 (-), C3.1, R4.2, SW1.2 (B), C1.2; no longer C3.2, R3.1
- net at J1.6 (EVN): now also J4.2 (Pin_2)
- net BATT_SENSE: now reaches R3.2
- net BATT_SENSE: now also C3.2, R4.1, U1.33 (41_A17); no longer R4.2
- net at R1.1, SW1.1 (A): now also Q1.1 (G)
- net at R1.2: now also BT2.1 (+), Q1.3 (S); no longer BT2.2 (-)
- net at J1.5 (ODD): now also J4.1 (Pin_1)
Other:
- moved on the sheet: BT2, R1, SW1

Commit message: started DPS
Parts:
- added HS1: Heatsink_Pad, Linefollower:Heatsink_HS-123-25_TO220_STONECOLD, symbol Mechanical:Heatsink_Pad
- C1: footprint (none) -> Capacitor_THT:C_Disc_D5.0mm_W2.5mm_P5.00mm
- C2: footprint (none) -> Capacitor_THT:CP_Radial_D6.3mm_P2.50mm
- C3: footprint (none) -> Capacitor_THT:C_Disc_D4.3mm_W1.9mm_P5.00mm
- R3, R4: footprint (none) -> Resistor_THT:R_Axial_DIN0204_L3.6mm_D1.6mm_P7.62mm_Horizontal
Connections:
- net GND: now also HS1.1
Changed lines of the file:
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@@
 	(wire
 		(pts
+			(xy 205.74 60.96) (xy 205.74 66.04)
+		)
+		(stroke
+			(width 0)
+			(type default)
+		)
+	)
+	(wire
+		(pts
 			(xy 81.28 146.05) (xy 81.28 93.98)
 		)
@@
 	)
 	(label "GND"
+		(at 205.74 66.04 0)
+		(effects
+			(font
+				(size 1.27 1.27)
+			)
+			(justify left bottom)
+		)
+	)
+	(label "GND"
 		(at 41.91 68.58 0)
 		(effects
@@
 			)
 		)
-		(property "Footprint" ""
+		(property "Footprint" "Resistor_THT:R_Axial_DIN0204_L3.6mm_D1.6mm_P7.62mm_Horizontal"
 			(at 240.03 90.678 90)
 			(effects
@@
 	)
 	(symbol
+		(lib_id "Mechanical:Heatsink_Pad")
+		(at 205.74 58.42 0)
+		(mirror y)
+		(unit 1)
+		(exclude_from_sim no)
+		(in_bom yes)
+		(on_board yes)
+		(dnp no)
+		(property "Reference" "HS1"
+			(at 201.93 56.5149 0)
+			(effects
+				(font
+					(size 1.27 1.27)
+				)
+				(justify left)
+			)
+		)
+		(property "Value" "Heatsink_Pad"
+			(at 201.93 59.0549 0)
+			(effects
+				(font
+					(size 1.27 1.27)
+				)
+				(justify left)
+			)
+		)
+		(property "Footprint" "Linefollower:Heatsink_HS-123-25_TO220_STONECOLD"
+			(at 205.4352 59.69 0)
+			(effects
+				(font
+					(size 1.27 1.27)
+				)
+				(hide yes)
+			)
+		)
+		(property "Datasheet" "~"
+			(at 205.4352 59.69 0)
+			(effects
+				(font
+					(size 1.27 1.27)
+				)
+				(hide yes)
+			)
+		)
+		(property "Description" "Heatsink with electrical connection, 1 pin"
+			(at 205.74 58.42 0)
+			(effects
+				(font
+					(size 1.27 1.27)
+				)
+				(hide yes)
+			)
+		)
+		(pin "1"
+		)
+		(instances
+			(project "LF_CB_modular_v1"
+				(path "/44d8d455-f542-4ff0-9bd6-aa534d2f06ad"
+					(reference "HS1")
+					(unit 1)
+				)
+			)
+		)
+	)
+	(symbol
 		(lib_id "Switch:SW_SPDT")
 		(at 242.57 123.19 180)
@@
 			)
 		)
-		(property "Footprint" ""
+		(property "Footprint" "Capacitor_THT:CP_Radial_D6.3mm_P2.50mm"
 			(at 234.95 49.8348 0)
 			(effects
@@
 			)
 		)
-		(property "Footprint" ""
+		(property "Footprint" "Capacitor_THT:C_Disc_D4.3mm_W1.9mm_P5.00mm"
 			(at 236.22 94.2848 0)
 			(effects
@@
 			)
 		)
-		(property "Footprint" ""
+		(property "Footprint" "Resistor_THT:R_Axial_DIN0204_L3.6mm_D1.6mm_P7.62mm_Horizontal"
 			(at 223.52 94.488 90)
 			(effects
@@
 		(on_board yes)
 		(dnp no)
-		(fields_autoplaced yes)
 		(property "Reference" "U2"
-			(at 213.36 57.1499 90)
+			(at 211.328 57.15 0)
 			(effects
 				(font
 					(size 1.27 1.27)
 				)
-				(justify left)
+				(justify right)
 			)
 		)
 		(property "Value" "LM7805_TO220"
-			(at 213.36 59.6899 90)
+			(at 213.36 51.308 0)
 			(effects
 				(font
 					(size 1.27 1.27)
 				)
-				(justify left)
+				(justify right)
 			)
 		)
@@
 			)
 		)
-		(property "Footprint" ""
+		(property "Footprint" "Capacitor_THT:C_Disc_D5.0mm_W2.5mm_P5.00mm"
 			(at 234.95 67.0052 0)
 			(effects

Commit message: power modul finishing
Parts:
- added C4, C5: C_100n, Capacitor_THT:C_Disc_D4.3mm_W1.9mm_P5.00mm, symbol Device:C
- added JW1, JW2: Cam_SCK, Linefollower:Jumper_pin, symbol Linefollower:Jumper_pin
- added JW3, JW4: 3V3, Linefollower:Jumper_pin, symbol Linefollower:Jumper_pin
- U2: value LM7805_TO220 -> LM2940CT-5.0 _TO220
Connections:
- net 3V3: now also JW4.1 (Pin_1); no longer J1.3 (VCC), J1.4 (VCC), U1.46 (3V3)
- net 5V: now also C5.2
- net 6V: now also C4.2
- net GND: now also C4.1, C5.1
- net Cam_SCK: no longer names the net of U1.35 (13_SCK_LED)
- net Cam_SCK: now also JW1.1 (Pin_1); no longer J2.3 (SCK)
- new net: J2.3 (SCK), JW2.1 (Pin_1)
- new net: J1.3 (VCC), J1.4 (VCC), JW3.1 (Pin_1)
- no-connect marks 21 -> 22
Other:
- moved on the sheet: C2, HS1, J4, U2

Commit message: getting ready for jlcpcb
Parts:
- removed JW1, JW2: Cam_SCK, Linefollower:Jumper_pin, symbol Linefollower:Jumper_pin
- removed JW3, JW4: 3V3, Linefollower:Jumper_pin, symbol Linefollower:Jumper_pin
- added U3: TSR_1-2433, Converter_DCDC:Converter_DCDC_TRACO_TSR-1_THT, symbol Converter_DCDC:TSR_1-2433
Connections:
- net 3V3: now also J1.3 (VCC), J1.4 (VCC), U3.3 (Vout); no longer U1.15 (3V3)
- net 6V: now also U3.1 (Vin)
- net GND: now also U3.2 (GND)
- net Cam_SCK: now reaches U1.35 (13_SCK_LED)
- net Cam_SCK: now also J2.3 (SCK)
- no-connect marks 22 -> 23
Other:
- moved on the sheet: BT2, C1, C2, C3, C4, C5, HS1, Q1, R1, R3, R4, SW1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

Commit message: added notes, sedond layer copper mask
Parts:
- added C6: C_Polarized_47u, Capacitor_THT:CP_Radial_D6.3mm_P2.50mm, symbol Device:C_Polarized
Connections:
- net 6V: now also C6.1
- net GND: now also C6.2
Changed lines of the file:
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@@
 	)
 	(junction
+		(at 45.72 50.8)
+		(diameter 0)
+		(color 0 0 0 0)
+	)
+	(junction
 		(at 220.98 96.52)
 		(diameter 0)
@@
 	(wire
 		(pts
+			(xy 45.72 39.37) (xy 45.72 50.8)
+		)
+		(stroke
+			(width 0)
+			(type default)
+		)
+	)
+	(wire
+		(pts
 			(xy 261.62 55.88) (xy 261.62 63.5)
 		)
@@
 	(wire
 		(pts
+			(xy 45.72 50.8) (xy 46.99 50.8)
+		)
+		(stroke
+			(width 0)
+			(type default)
+		)
+	)
+	(wire
+		(pts
 			(xy 156.21 88.9) (xy 149.86 88.9)
 		)
@@
 	(wire
 		(pts
-			(xy 41.91 50.8) (xy 46.99 50.8)
+			(xy 41.91 50.8) (xy 45.72 50.8)
 		)
 		(stroke
@@
 		)
 	)
+	(label "GND"
+		(at 45.72 31.75 0)
+		(effects
+			(font
+				(size 1.27 1.27)
+			)
+			(justify left bottom)
+		)
+	)
 	(label "3V3"
 		(at 148.59 156.21 0)
@@
 					(unit 1)
 				)
+			)
+		)
+	)
+	(symbol
+		(lib_id "Device:C_Polarized")
+		(at 45.72 35.56 180)
+		(unit 1)
+		(exclude_from_sim no)
+		(in_bom yes)
+		(on_board yes)
+		(dnp no)
+		(property "Reference" "C6"
+			(at 38.1 36.449 90)
+			(effects
+				(font
+					(size 1.27 1.27)
+				)
+			)
+		)
+		(property "Value" "C_Polarized_47u"
+			(at 40.64 36.449 90)
+			(effects
+				(font
+					(size 1.27 1.27)
+				)
+			)
+		)
+		(property "Footprint" "Capacitor_THT:CP_Radial_D6.3mm_P2.50mm"
+			(at 44.7548 31.75 0)
+			(effects
+				(font
+					(size 1.27 1.27)
+				)
+				(hide yes)
+			)
+		)
+		(property "Datasheet" "~"
+			(at 45.72 35.56 0)
+			(effects
+				(font
+					(size 1.27 1.27)
+				)
+				(hide yes)
+			)
+		)
+		(property "Description" "Polarized capacitor"
+			(at 45.72 35.56 0)
+			(effects
+				(font
+					(size 1.27 1.27)
+				)
+				(hide yes)
+			)
+		)
+		(pin "2"
+		)
+		(pin "1"
+		)
+		(instances
+			(project "LF_CB_modular_v1"
+				(path "/44d8d455-f542-4ff0-9bd6-aa534d2f06ad"
+					(reference "C6")
+					(unit 1)
+				)
