File: LF_4.0 - 26nat/KiCad/LF_CB_modular_v1/LF_CB_modular_v1.kicad_sch (KiCad schematic)
At the start: 28 parts, among them J1 Conn_QTR16, J10 Conn_01x02, J11 Conn_01x10, J2 Conn_Arducam_MEGA_3mpx, J3 Conn_TB6612FNG_IC, J4 Conn_01x02, J8 Conn_01x01, J9 Conn_01x01, M1 Motor_DC, M2 Motor_DC, Q1 IRF4905, SW1 SW_SPDT, U1 Teensy4.1, U2 LM2940CT-5.0 _TO220, U3 TSR_1-2433

Commit message: replaced XT60 by wire
Parts:
- BT2: footprint Connector_AMASS:AMASS_XT60PW-M_1x02_P7.20mm_Horizontal -> Connector_Wire:SolderWire-2sqmm_1x02_P7.8mm_D2mm_OD3.9mm
Changed lines of the file:
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@@
 			)
 		)
-		(property "Footprint" "Connector_AMASS:AMASS_XT60PW-M_1x02_P7.20mm_Horizontal"
+		(property "Footprint" "Connector_Wire:SolderWire-2sqmm_1x02_P7.8mm_D2mm_OD3.9mm"
 			(at 246.126 147.32 90)
 			(effects

Commit message: final. hope so
Parts:
- added J5, J6: Conn_01x05, Connector_PinSocket_2.54mm:PinSocket_1x05_P2.54mm_Vertical, symbol Connector_Generic:Conn_01x05
Connections:
- net GND: now also J5.1 (Pin_1), J5.2 (Pin_2), J5.3 (Pin_3), J5.4 (Pin_4), J5.5 (Pin_5), J6.1 (Pin_1), J6.2 (Pin_2), J6.3 (Pin_3), J6.4 (Pin_4), J6.5 (Pin_5)
